File: hardware/kicad/bluetooth-speaker.kicad_sch (KiCad schematic)
At the start: 14 parts, among them U1 ESP32-WROOM-32E, U2 TAS5805MPWP

Commit message: IC Selection WiP
Parts:
- added C13, C17, C18, C19, C20: 10u, symbol Device:C_Small
- added C14, C15, C21, C23: 100n, symbol Device:C_Small
- added C16: 4.7u, symbol Device:C_Small
- added C22: 2.2u, symbol Device:C_Small
- added C24, C25, C26: 22u, symbol Device:C_Small
- added J?: USB_C_Receptacle_USB2.0_16P, Connector_USB:USB_C_Receptacle_GCT_USB4105-xx-A_16P_TopMnt_Horizontal, symbol Connector:USB_C_Receptacle_USB2.0_16P
- added L?: 2.2u, 8A, symbol Device:L_Small
- added L?: 2.2u, symbol Device:L_Small
- added R1, R2, R3, R?: 22, symbol Device:R_Small_US
- added R10: 18k, symbol Device:R_Small_US
- added R11, R12, R13, R9: 100k, symbol Device:R_Small_US
- added R4, R5, R6, R7: 4.7k, symbol Device:R_Small_US
- added R8: 100, symbol Device:R_Small_US
- added TP1, TP2, TP3, TP?: TestPoint, symbol Connector:TestPoint
- added U?: TPS63001, Package_SON:Texas_DRC0010J_ThermalVias, symbol Regulator_Switching:TPS63001
- added U?: BQ24075RGT, Package_DFN_QFN:VQFN-16-1EP_3x3mm_P0.5mm_EP1.6x1.6mm, symbol Battery_Management:BQ24075RGT
- added U?: CP2102N-Axx-xQFN20, Package_DFN_QFN:SiliconLabs_QFN-20-1EP_3x3mm_P0.5mm, symbol Interface_USB:CP2102N-Axx-xQFN20
- added U?: TPS61089, Package_DFN_QFN:Texas_VQFN-RNR0011A-11, symbol Regulator_Switching:TPS61089
Connections:
- net at C5.1, U2.13 (AVDD): no longer C12.1
- net AMP_FAULT: now reaches U1.13 (IO14)
- net AMP_FAULT: now also U2.3 (ADR/~{FAULT}), R4.1
- net AMP_PDNb: now reaches U1.16 (IO13)
- net AMP_PDNb: now also U2.12 (~{PDN}), R5.1
- net PWR_3V3: now reaches U1.2 (VDD)
- net PWR_3V3: now also U1.3 (EN), U2.2 (DVDD), C13.1, C14.1, C15.1, C16.1, C19.1, R4.2, R5.2, R6.2, R7.2, U?.1 (VOUT), U?.10 (FB)
- net at U1.24 (IO2): now also R1.1
- net at U1.25 (IO0): now also R?.1
- net at U1.26 (IO4): now also R2.1
- net I2C_SCL: now reaches U1.27 (IO16)
- net I2C_SCL: now also U2.11 (SCL), R7.1
- net I2C_SDA: now reaches U1.28 (IO17)
- net I2C_SDA: now also U2.10 (SDA), R6.1
- net I2S_SDOUT: now reaches U1.29 (IO5)
- net I2S_SDOUT: now also R3.1, TP3.1
- net at U2.4 (VR_DIG): now also C12.1
- net I2S_LRCLK: now reaches U2.6 (LRCLK)
- net I2S_LRCLK: now also R1.2, TP1.1
- net I2S_SCLK: now reaches U2.7 (SCLK)
- net I2S_SCLK: now also R?.2, TP?.1
- net I2S_SDIN: now reaches U2.8 (SDIN)
- net I2S_SDIN: now also R2.2, TP2.1
- net at U2.9 (SDOUT): now also R3.2
- net 8V_PVDD renamed PWR_8V_PVDD
- net PWR_8V_PVDD: now also C24.1, C25.2, C26.2, R11.1, U?.6 (VOUT)
- new net: C24.2, C25.1, C26.1
- new net: C13.2, C19.2
- new net: C18.1, R8.1, U?.6 (EN), U?.7 (PS/SYNC), U?.8 (VINA)
- new net: C20.2, C21.2
- new net: J?.A1 (GND), J?.A12 (GND), J?.B1 (GND), J?.B12 (GND)
- new net: J?.A4 (VBUS), J?.A9 (VBUS), J?.B4 (VBUS), J?.B9 (VBUS)
- new net: R9.1, U?.1 (FSW)
- new net: U?.11 (PGND), U?.3 (PGND), U?.9 (GND)
- new net: L?.1, U?.2 (L2)
- new net: L?.2, U?.4 (L1)
- new net: R10.1, R11.2, U?.3 (FB)
- new net: L?.2, U?.11 (SW)
- new net: U?.10 (OUT), U?.11 (OUT)
- new net: U?.17 (VSS), U?.8 (VSS)
- new net: U?.2 (BAT), U?.3 (BAT)
- new net: C23.2, U?.10 (BOOT)
- new net: R12.2, R13.1
- new net: U?.12 (GND), U?.21 (GND), U?.3 (GND)
- new net: C22.1, U?.2 (VCC)
- new net: R12.1, U?.8 (ILIM)
- new net PWR_IN_5V: C17.1, C20.1, C21.1, C23.1, L?.1, R8.2, R9.2, U?.5 (VIN), U?.7 (EN), U?.9 (VIN)
Other:
- note added: "I2C Address: 0101100"
- moved on the sheet: C1, C10, C11, C12, C2, C3, C4, C5, C6, C7, C8, C9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
