File: hardware/kicad/bluetooth-speaker.kicad_sch (KiCad schematic)
At the start: 53 parts, among them U1 ESP32-WROOM-32E, U2 TAS5805MPWP

Commit message: IC selection WiP
Parts:
- removed C8, C9: 220n, symbol Device:C_Small
- added C27, C30, C31: 100n, symbol Device:C_Small
- added C28: 10u, symbol Device:C_Small
- added C29, C32: 4.7u, symbol Device:C_Small
- added C33: 22u, symbol Device:C_Small
- added C?: 10n, symbol Device:C_Small
- added D?: LED, symbol Device:LED
- added J?: Conn_01x02_Pin, symbol Connector:Conn_01x02_Pin
- added R14, R?: 5.1k, symbol Device:R_Small_US
- added R?: 0, symbol Device:R_Small_US
Connections:
- net PWR_3V3: now also U?.6 (VDD), U?.7 (VREGIN), U?.8 (VBUS), C29.1, C30.1, C31.1, C32.1
- net at J?.A1 (GND), J?.A12 (GND), J?.B1 (GND)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: now also C?.2, R?.2
- net USB_VBUS: now reaches J?.A4 (VBUS), J?.A9 (VBUS), J?.B4 (VBUS), J?.B9 (VBUS)
- net USB_VBUS: now also U?.13 (IN), C27.1, C28.1
- net at J?.A5 (CC1): now also R?.1
- net USB_DP: now reaches J?.A6 (D+)
- net USB_DP: now also J?.B6 (D+), U?.4 (D+)
- net USB_DN: now reaches J?.A7 (D-)
- net USB_DN: now also J?.B7 (D-), U?.5 (D-)
- net at J?.B5 (CC2): now also R14.1
- net at J?.S1 (SHIELD): now also C?.1, R?.1
- net VBAT_MONITOR: now reaches U1.4 (SENSOR_VP)
- net DRIVER_N: now reaches C7.1, U2.23 (OUT_A-)
- net DRIVER_N: now also J?.2 (Pin_2)
- net DRIVER_P: now reaches C6.2, U2.26 (OUT_A+)
- net DRIVER_P: now also J?.1 (Pin_1)
- net PWR_PATH_OUT: now reaches U?.10 (OUT), U?.11 (OUT)
- net PWR_PATH_OUT: now also D?.2 (A)
- net VBAT_P: now reaches U?.2 (BAT), U?.3 (BAT)
- net VBAT_P: now also C33.1
- net at U?.9 (~{CHG}): now also D?.1 (K)
- no-connect marks 0 -> 7
